Commit message: add X and Y translation

File: robot_description/urdf/robot.xacro (robot description, xacro)
@@ -17,12 +17,24 @@
   <link name="world"/>
   <joint name="fixed" type="fixed">
-        <origin xyz="0 0 0.01" rpy="0 0 0"/>
+        <origin xyz="0 0 0.0" rpy="0 0 0"/>
         <parent link="world"/>
         <child link="base_link"/>
   </joint>
-<!--     <link name="X_base_link"/>   -->
-<!--     <link name="Y_base_link"/>   -->
+    <link name="X_base_link">
+        <inertial>
+            <origin xyz="0 0 0" rpy="0 0 0"/>
+            <mass value="0.01"/>
+            <box_inertia m="0.01" x="0.02" y="0.02" z="0.05"/>
+        </inertial>
+    </link>
+    <link name="Y_base_link">
+        <inertial>
+            <origin xyz="0 0 0" rpy="0 0 0"/>
+            <mass value="0.01"/>
+            <box_inertia m="0.01" x="0.02" y="0.02" z="0.05"/>
+        </inertial>
+    </link>
     <link name="base_link">
-        <visual>
+<!--        <visual>
             <geometry>
                 <cylinder length="0.01" radius=".053" />
@@ -30,5 +42,5 @@
             <material name="black" />
             <origin rpy="0 0 0" xyz="0 0 0" />
-        </visual>
+        </visual>     -->
         <inertial>
             <origin xyz="0 0 0" rpy="0 0 0"/>
@@ -201,7 +213,7 @@
         </collision>
     </link>
-<!--    <joint name="X_base_joint" type="prismatic">
-        <axis xyz="1 0 0" />
-        <limit effort="1000.0" lower="-5.0" upper="5.0" velocity="1.0" />
+    <joint name="X_base_joint" type="prismatic">
+        <axis xyz="1 0 0" />
+        <limit effort="100.0" lower="-5.0" upper="5.0" velocity="1.0" />
         <origin rpy="0 0 0" xyz="0 0 0" />
         <parent link="base_link" />
@@ -210,15 +222,14 @@
     <joint name="Y_base_joint" type="prismatic">
         <axis xyz="0 1 0" />
-        <limit effort="1000.0" lower="-5.0" upper="5.0" velocity="1.0" />
+        <limit effort="100.0" lower="-5.0" upper="5.0" velocity="1.0" />
         <origin rpy="0 0 0" xyz="0 0 0" />
         <parent link="X_base_link" />
         <child link="Y_base_link" />
-    </joint>-->
+    </joint>
     <joint name="base_joint" type="revolute">
         <axis xyz="0 0 1" />
         <limit effort="1000.0" lower="0.0" upper="3.1416" velocity="1.0" />
         <origin rpy="0 0 0" xyz="0 0 0" />
-        <!--<parent link="Y_base_link" />-->
-        <parent link="base_link" />
+        <parent link="Y_base_link" />
         <child link="robot_base_link" />
     </joint>

Commit message: ready to create challenges

File: robot_description/urdf/robot.xacro (robot description, xacro)
@@ -36,11 +36,4 @@
     </link>
     <link name="base_link">
-<!--        <visual>
-            <geometry>
-                <cylinder length="0.01" radius=".053" />
-            </geometry>
-            <material name="black" />
-            <origin rpy="0 0 0" xyz="0 0 0" />
-        </visual>     -->
         <inertial>
             <origin xyz="0 0 0" rpy="0 0 0"/>
@@ -153,12 +146,12 @@
             </geometry>
             <material name="black" />
-            <origin rpy="0 -1.5708 0" xyz="0 0 -0.025" />
-        </collision>
-        <visual>
-            <geometry>
-                <box size="0.05 0.02 0.01"/>
-            </geometry>
-            <material name="black" />
-            <origin rpy="0 -1.5708 0" xyz="0 0 -0.025" />
+            <origin rpy="0 -1.570808 0" xyz="0 0 -0.025" />
+        </collision>
+        <visual>
+            <geometry>
+                <box size="0.05 0.02 0.01"/>
+            </geometry>
+            <material name="black" />
+            <origin rpy="0 -1.570808 0" xyz="0 0 -0.025" />
         </visual>
         <inertial>
@@ -174,12 +167,12 @@
             </geometry>
             <material name="black" />
-            <origin rpy="0 -1.5708 0" xyz="0 0 -0.025" />
-        </collision>
-        <visual>
-            <geometry>
-                <box size="0.05 0.02 0.01"/>
-            </geometry>
-            <material name="black" />
-            <origin rpy="0 -1.5708 0" xyz="0 0 -0.025" />
+            <origin rpy="0 -1.570808 0" xyz="0 0 -0.025" />
+        </collision>
+        <visual>
+            <geometry>
+                <box size="0.05 0.02 0.01"/>
+            </geometry>
+            <material name="black" />
+            <origin rpy="0 -1.570808 0" xyz="0 0 -0.025" />
         </visual>
         <inertial>
@@ -229,5 +222,5 @@
     <joint name="base_joint" type="revolute">
         <axis xyz="0 0 1" />
-        <limit effort="1000.0" lower="0.0" upper="3.1416" velocity="1.0" />
+        <limit effort="1000.0" lower="-3.1416" upper="3.1416" velocity="1.0" />
         <origin rpy="0 0 0" xyz="0 0 0" />
         <parent link="Y_base_link" />
@@ -237,5 +230,5 @@
         <axis xyz="1 0 0" />
         <limit effort="1000.0" lower="0.2618" upper="2.8798" velocity="1.0" />
-        <origin rpy="-1.5708 0 0" xyz="0 -.002 0.072" />
+        <origin rpy="-1.570808 0 0" xyz="0 -.002 0.072" />
         <parent link="robot_base_link" />
         <child link="shoulder_link" />
@@ -244,5 +237,5 @@
         <axis xyz="1 0 0" />
         <limit effort="1000.0" lower="0" upper="3.1416" velocity="1.0" />
-        <origin rpy="-1.5708 0 0" xyz="0 0 0.125" />
+        <origin rpy="-1.570808 0 0" xyz="0 0 0.125" />
         <parent link="shoulder_link" />
         <child link="elbow_link" />
@@ -251,5 +244,5 @@
         <axis xyz="1 0 0" />
         <limit effort="1000.0" lower="0" upper="3.1416" velocity="1.0" />
-        <origin rpy="-1.5708 0 0" xyz="0 0 0.125" />
+        <origin rpy="-1.570808 0 0" xyz="0 0 0.125" />
         <parent link="elbow_link" />
         <child link="wrist_pitch_link" />
@@ -258,5 +251,5 @@
         <axis xyz="0 0 -1" />
         <limit effort="1000.0" lower="0" upper="3.1416" velocity="1.0" />
-        <origin rpy="0 0 1.5708" xyz="0 0.0 0.06" />
+        <origin rpy="0 0 1.570808" xyz="0 0.0 0.06" />
         <parent link="wrist_pitch_link" />
         <child link="wrist_roll_link" />
@@ -278,6 +271,6 @@
     </joint>
     <joint name="camera_joint" type="fixed">
-        <origin xyz="0 0.04 0" rpy="-1.57 -1.57 0" />
-        <parent link="wrist_roll_link" />
+        <origin xyz="0 0 0.8" rpy="1.5708 1.5708 -1.5708" />
+        <parent link="robot_base_link" />
         <child link="camera_embedded_link"/>
     </joint>
