Commit message: can add box and obstacle

File: robotics_challenges/urdf/cube.xacro (robot description, xacro)
@@ -3,8 +3,8 @@
     <xacro:arg name="id" default="1" />
     <xacro:include filename="$(find robotics_challenges)/urdf/cube_marker.xacro" />
-    <link name="my_box">
+    <link name="my_cube$(arg id)">
         <aruco_cube id="$(arg id)" dim="0.05" m="0.05"/>
     </link>
-    <gazebo reference="my_box">
+    <gazebo reference="my_cube$(arg id)">
     <mu1>100.0</mu1>
     <mu2>100.0</mu2>

File: robotics_challenges/urdf/obstacle.xacro (robot description, xacro)
@@ -1,27 +1,14 @@
 <?xml version="1.0"?>
 <robot xmlns:xacro="http://www.ros.org/wiki/xacro">
-    <xacro:property name="num_marker" value="0" />
-    <xacro:property name="dim" value="1.0" />
-    <xacro:property name="m" value="100" />
-<!--  <xacro:macro name="aruco_cube" params="num_marker dim m ">  -->
-<link name="obstacle">
-   <inertial>
-      <origin xyz="0 0 0" />
-      <mass value="${m}" />
-      <inertia  ixx="${m*m/12.0}" ixy="0.0"  ixz="0.0"  iyy="${m*m/12.0}"  iyz="0.0"  izz="${m*m/12.0}" />
-    </inertial>
-    <visual>
-      <geometry>
-        <box size="${dim} ${dim*0.1} ${dim*0.15}" />
-      </geometry>
-    </visual>
-    <collision>
-      <geometry>
-        <box size="${dim} ${dim*0.1} ${dim*0.15}" />
-      </geometry>
-    </collision>
-<!-- </xacro:macro>      -->
-</link>
-    <gazebo reference="obstacle">
+    <xacro:arg name="id" default="1" />
+    <xacro:arg name="dim" default="0.05" />
+    <xacro:arg name="r" default="0.05" />
+    <xacro:arg name="h" default="0.1" />
+    <xacro:arg name="m" default="0.05" />
+    <xacro:include filename="$(find robotics_challenges)/urdf/obstacle_marker.xacro" />
+    <link name="my_obstacle$(arg id)">
+        <obstacle id="$(arg id)" dim="$(arg dim)" r="$(arg r)" h="$(arg h)" m="$(arg m)"/>
+    </link>
+    <gazebo reference="my_obstacle$(arg id)">
     <mu1>100.0</mu1>
     <mu2>100.0</mu2>
