Commit message: ready for the challenges

File: robotics_challenges/urdf/box_marker.xacro (robot description, xacro)
@@ -44,5 +44,5 @@
     </visual>
     <collision>
-      <origin xyz="${l/2} ${l/2} ${width/2}" rpy="0 0 0"/>
+      <origin xyz="0 0 ${width/2}" rpy="0 0 0"/>
       <geometry>
         <box size="${l} ${l} ${width}" />
